Commit message: Remove inertia of root link -> Fix warning

File: urdf/psen_scan.urdf.xacro (robot description, xacro)
@@ -12,12 +12,5 @@
     <xacro:property name="dist_scanning_axis_rear" value="0.0525" /> <!-- src datasheet p 96 -->
     <!-- Location of mounting point at the lower back of device -->
-    <link name="${prefix}_mount_link">
-      <inertial>
-        <mass value="0.001" />
-        <origin xyz="0 0 0" />
-        <inertia ixx="0.000001" ixy="0.0" ixz="0.0"
-          iyy="0.000001" iyz="0.0" izz="0.000001" /> <!-- TODO correct dimensions -->
-      </inertial>
-    </link>
+    <link name="${prefix}_mount_link"/>
     <joint name="${prefix}_mount_joint" type="fixed">
       <parent link="${prefix}_mount_link" />

Commit message: Move mounting between screw holes

File: urdf/psen_scan.urdf.xacro (robot description, xacro)
@@ -16,5 +16,5 @@
       <parent link="${prefix}_mount_link" />
       <child link="${prefix}" />
-      <origin rpy="0 0 0" xyz="${radius} 0 ${height / 2}"/>
+      <origin rpy="0 0 0" xyz="${radius} 0 0"/>
     </joint>
     <!-- Location of scanner body -->

Commit message: correct height and moments of inertia in xacro

File: urdf/psen_scan.urdf.xacro (robot description, xacro)
@@ -16,5 +16,5 @@
       <parent link="${prefix}_mount_link" />
       <child link="${prefix}" />
-      <origin rpy="0 0 0" xyz="${radius} 0 0"/>
+      <origin rpy="0 0 0" xyz="${radius} 0 ${height / 2}"/>
     </joint>
     <!-- Location of scanner body -->
@@ -22,5 +22,5 @@
       <visual>
         <geometry>
-            <cylinder radius="${radius}" length="${height}" />
+          <cylinder radius="${radius}" length="${height}" />
         </geometry>
         <material name="pilz_yellow" >
@@ -30,5 +30,5 @@
       <collision>
         <geometry>
-            <cylinder radius="${radius}" length="${height}" />
+          <cylinder radius="${radius}" length="${height}" />
         </geometry>
       </collision>
@@ -36,7 +36,7 @@
         <mass value="${mass}" />
         <origin xyz="0 0 0" />
-        <inertia ixx="${0.0833333 * mass * (radius * radius + height * height)}" ixy="0.0" ixz="0.0"
-          iyy="${0.0833333 * mass * (radius * radius + height * height)}" iyz="0.0"
-          izz="${0.0833333 * mass * (radius * radius + radius * radius)}" /> <!-- TODO correct dimensions -->
+        <inertia ixx="${1 / 12 * mass * (3 * radius * radius + height * height)}" ixy="0.0" ixz="0.0"
+          iyy="${1 / 12 * mass * (3 * radius * radius + height * height)}" iyz="0.0"
+          izz="${.5 * mass * (radius * radius)}" />
       </inertial>
     </link>

Commit message: taking review comments into account

File: urdf/psen_scan.urdf.xacro (robot description, xacro)
@@ -2,8 +2,4 @@
 <robot xmlns:xacro="http://ros.org/wiki/xacro">
   <xacro:macro name="psen_scan" params="prefix">
-    <xacro:property name="min_range" value="0.1" /> <!-- TODO correct dimensions -->
-    <xacro:property name="max_range" value="4.0" /> <!-- TODO correct dimensions -->
-    <xacro:property name="min_angle" value="$(eval -137.5 /180.0 * pi)" /> <!-- src datasheet p 91 -->
-    <xacro:property name="max_angle" value="$(eval 137.5 /180.0 * pi)" /> <!-- src datasheet p 91 -->
     <xacro:property name="mass" value="1.53" /> <!-- src datasheet p 96 -->
     <xacro:property name="radius" value="0.051" /> <!-- src datasheet p 96 -->

Commit message: trying meshes

File: urdf/psen_scan.urdf.xacro (robot description, xacro)
@@ -18,5 +18,6 @@
       <visual>
         <geometry>
-          <cylinder radius="${radius}" length="${height}" />
+          <!-- <cylinder radius="${radius}" length="${height}" /> -->
+          <mesh filename="package://psen_scan_v2/meshes/psenscan_smaller.stl" />
         </geometry>
         <material name="pilz_yellow" >
