Commit message: update zonSet markers visualization and compability with one scanner, two, three, four

File: urdf/main.urdf.xacro (robot description, xacro)
@@ -1,26 +1,35 @@
 <?xml version="1.0"?>
 <robot xmlns:xacro="http://ros.org/wiki/xacro" name="psen_scan">
-  <!-- Example on how to use the psen_scan scanner within your robots urdf -->
+  <!-- PSENscan arguments -->
+  <xacro:arg name="nr_scanners" default="0"/>
   <xacro:arg name="prefix" default="laser_1"/>
-  <xacro:arg name="prefix_0" default="laser_1_Subscriber0"/>
-  <!-- <xacro:arg name="prefix_1" default="laser_1_Subscriber1"/> -->
-  <!-- <xacro:arg name="prefix_2" default="laser_1_Subscriber2"/> -->
+  <xacro:arg name="prefix_sub0" default="laser_1_Subscriber0"/>
+  <xacro:arg name="prefix_sub1" default="laser_1_Subscriber1"/>
+  <xacro:arg name="prefix_sub2" default="laser_1_Subscriber2"/>
+  <!-- Number of Subscribers -->
+  <xacro:property name="nr_sub" value="$(arg nr_scanners)"/>
   <xacro:include filename="$(find psen_scan_v2)/urdf/xacros/psen_scan.urdf.xacro" />
   <link name="base_link"/>
   <!-- PSENscan Master -->
   <xacro:psen_scan prefix="$(arg prefix)" parent="base_link">
-    <origin xyz="0 0 0" rpy="0 0 0" />
+    <origin xyz="0.5 0 0" rpy="0 0 0" />
   </xacro:psen_scan>
   <!-- PSENscan Subscriber0 -->
-  <xacro:psen_scan prefix="$(arg prefix_0)" parent="base_link">
-    <origin xyz="-0.5 0 0" rpy="0 0 3.14" />
-  </xacro:psen_scan>
+  <xacro:if value="${nr_sub >= 1}">
+    <xacro:psen_scan prefix="$(arg prefix_sub0)" parent="base_link">
+      <origin xyz="-0.5 0 0" rpy="0 0 3.14" />
+    </xacro:psen_scan>
+  </xacro:if>
   <!-- PSENscan Subscriber1 -->
-  <!-- <xacro:psen_scan prefix="$(arg prefix_1)" parent="base_link">
-    <origin xyz="-0.5 0.5 0" rpy="0 0 3.14" />
-  </xacro:psen_scan> -->
+  <xacro:if value="${nr_sub >= 2}">
+    <xacro:psen_scan prefix="$(arg prefix_sub1)" parent="base_link">
+      <origin xyz="0 0.5 0" rpy="0 0 1.57" />
+    </xacro:psen_scan>
+  </xacro:if>
   <!-- PSENscan Subscriber2 -->
-  <!-- <xacro:psen_scan prefix="$(arg prefix_2)" parent="base_link">
-    <origin xyz="0.5 -0.5 0" rpy="0 0 3.14" />
-  </xacro:psen_scan> -->
+  <xacro:if value="${nr_sub == 3}">
+    <xacro:psen_scan prefix="$(arg prefix_sub2)" parent="base_link">
+      <origin xyz="0 -0.5 0" rpy="0 0 -1.57" />
+    </xacro:psen_scan>
+  </xacro:if>
 </robot>

Commit message: update code optimization

File: urdf/main.urdf.xacro (robot description, xacro)
@@ -10,12 +10,12 @@
   <xacro:property name="nr_sub" value="$(arg nr_scanners)"/>
   <xacro:include filename="$(find psen_scan_v2)/urdf/xacros/psen_scan.urdf.xacro" />
-  <link name="base_link"/>
+  <link name="reference_link"/>
   <!-- PSENscan Master -->
-  <xacro:psen_scan prefix="$(arg prefix)" parent="base_link">
+  <xacro:psen_scan prefix="$(arg prefix)" parent="reference_link">
     <origin xyz="0.5 0 0" rpy="0 0 0" />
   </xacro:psen_scan>
   <!-- PSENscan Subscriber0 -->
   <xacro:if value="${nr_sub >= 1}">
-    <xacro:psen_scan prefix="$(arg prefix_sub0)" parent="base_link">
+    <xacro:psen_scan prefix="$(arg prefix_sub0)" parent="reference_link">
       <origin xyz="-0.5 0 0" rpy="0 0 3.14" />
     </xacro:psen_scan>
@@ -23,5 +23,5 @@
   <!-- PSENscan Subscriber1 -->
   <xacro:if value="${nr_sub >= 2}">
-    <xacro:psen_scan prefix="$(arg prefix_sub1)" parent="base_link">
+    <xacro:psen_scan prefix="$(arg prefix_sub1)" parent="reference_link">
       <origin xyz="0 0.5 0" rpy="0 0 1.57" />
     </xacro:psen_scan>
@@ -29,5 +29,5 @@
   <!-- PSENscan Subscriber2 -->
   <xacro:if value="${nr_sub == 3}">
-    <xacro:psen_scan prefix="$(arg prefix_sub2)" parent="base_link">
+    <xacro:psen_scan prefix="$(arg prefix_sub2)" parent="reference_link">
       <origin xyz="0 -0.5 0" rpy="0 0 -1.57" />
     </xacro:psen_scan>

File: urdf/xacros/psen_scan.urdf.xacro (robot description, xacro)
@@ -8,5 +8,5 @@
     <xacro:property name="dist_scanning_axis_rear" value="0.0525" /> <!-- src datasheet p 96 -->
     <joint name="${prefix}_joint" type="fixed">
-      <parent link="base_link" />
+      <parent link="reference_link" />
       <child link="${prefix}_mount_link" />
       <xacro:insert_block name="origin" />
